Commit message: Huge modifications and amazing results

File: wang/robot_assets/KR16_L6.urdf (robot description, URDF)
Before this commit: robot kr16_l6, 7 links, 6 joints
Joints:
- joint joint_1: limit lower=3.228859 upper=-3.228859 effort=300 velocity=3 -> lower=-3.228859 upper=3.228859 effort=300 velocity=3
- joint joint_2: limit lower=2.18166 upper=-1.1344 effort=300 velocity=3 -> lower=-1.1344 upper=2.18166 effort=300 velocity=3
- joint joint_3: limit lower=1.117 upper=-3.8397 effort=300 velocity=3 -> lower=-3.8397 upper=1.117 effort=300 velocity=3
